File: Electronics/Motherboard_simple.sch (EAGLE design)
At the start: 53 parts, among them IC1 NE556D, IC2 741G3157DBVR, IC3 741G3157DBVR, IC4 TINY25, J1 AVRISP, Q1 2N3904, Q2 2N3904, U2 USD-SOCKETNEW

Commit message: Moved RC Mux to subdirectory. Minor changes to various other boards.
Parts:
- removed IC1: NE556D, linear:NE556D
- removed IC2, IC3: 741G3157DBVR, 74xx-little-us:741G3157DBVR
- removed IC4: TINY25, avr-7:TINY138P3
- removed J1: AVRISP, ads4:AVRISP6
- removed JP16, JP18, JP23: POWER, pinhead-2:PINHD-1X02_2.54-S
- removed JP19: ENCODERS, pinhead-2:PINHD-1X03_2.54-S
- removed JP20: I2C, pinhead-2:PINHD-1X04_2.54-S
- removed JP21: RXE, pinhead-2:PINHD-1X03_2.54-S
- removed JP22: RXS, pinhead-2:PINHD-1X03_2.54-S
- removed JP7: PPS, pinhead-2:PINHD-1X01_2.54-S
- removed LED_L, LED_R: (no value), led:LED3MM
- removed Q1, Q2: 2N3904, mes_transistors:2N3904
- removed R11, R12, R15: 10k, rcl:R-US_0204/5
- removed R13, R14: 1k, rcl:R-US_0204/5
- removed R7, R8: 330, rcl:R-US_0204/5
- removed SJ1, SJ2: (no value), SparkFun:SOLDERJUMPER_2WAYS
- added C3: 10uF, rcl:CPOL-USE2.5-6
- added C4: 0.01uF, rcl:C-US050-025X075
- C1: value 104 -> 470uF; device rcl:C-US050-025X075 -> rcl:CPOL-USE2.5-6
- C2: value 104 -> 0.01uF
- JP15: device pinhead-2:PINHD-1X03_2.54-S -> pinhead-2:PINHD-1X04_2.54-S
- JP8: value ESC -> SPEED
- JP9: value SRV -> STEER
Connections:
- removed net !TRST: IC4.(RESET)PB5, J1.!RESET, R15.1
- removed net BEC: JP21.2, JP22.2, JP8.2, JP9.2
- removed net ESC: IC2G$1.X, JP8.1
- removed net MCUESC: IC2G$1.B, MBED.P22
- removed net MCUSRV: IC3G$1.B, MBED.P21
- removed net MCU_LEFT: IC1A.Q, LED_L.A, MBED.P30
- removed net MCU_RIGHT: IC1B.Q, LED_R.A, MBED.P29
- removed net MISO: IC4.(MISO)PB1, J1.MISO
- removed net N$11: IC1B.THR, IC1B.TR, Q2.C, R12.1
- removed net N$12: IC1A.THR, IC1A.TR, Q1.C, R11.1
- removed net N$13: Q2.B, R13.1
- removed net N$14: Q1.B, R14.1
- removed net N$18: JP10.1, SJ1.2
- removed net N$19: JP6.1, SJ2.2
- removed net N$25: IC2G$1.!A!/B, IC3G$1.!A!/B, IC4.(ADC3)PB3
- removed net N$4: LED_R.C, R8.2
- removed net PPS: JP7.1, MBED.P11
- removed net RXESC: IC2G$1.A, IC4.(MOSI)PB0, J1.MOSI, JP21.1, MBED.P24
- removed net RXSRV: IC3G$1.A, JP22.1, MBED.P23
- removed net SCK: IC4.(SCK)PB2, J1.SCK
- removed net SRV: IC3G$1.X, JP9.1
- new net SPEED: JP8.1, MBED.P22
- new net STEER: JP9.1, MBED.P21
- net +3V3: now also JP15.1; no longer C1.1, C2.1, IC1A.R, IC1A.V+, IC1B.R, IC4.VCC, J1.VCC, JP15.2, JP19.2, JP20.1, R11.2, R12.2, R15.2, SJ1.3, SJ2.3
- net +5V: now also C1.+, C2.1, C3.+, C4.1, JP10.1, JP6.1; no longer JP16.1, JP18.1, JP23.1, SJ1.1, SJ2.1
- net ENC_LEFT: now also JP15.2, MBED.P30; no longer JP15.1, R14.2
- net ENC_RIGHT: now also JP15.3, MBED.P29; no longer JP19.1, R13.2
- net GND: now also C1.-, C3.-, C4.2, JP15.4; no longer C1.2, IC1A.GND, IC4.GND, J1.GND, JP15.3, JP16.2, JP18.2, JP19.3, JP20.4, JP21.3, JP22.3, JP23.2, Q1.E, Q2.E, R7.1, R8.1
- net N$3: now also JP8.2, JP9.2; no longer LED_L.C, R7.2
- net N$5: now also JP1.2, MBED.P14; no longer JP1.4, MBED.P13
- net N$7: now also JP1.4, MBED.P15; no longer JP1.2, MBED.P12
- net N$8: now also MBED.P16; no longer MBED.P14
- net SCL: no longer JP20.3
- net SDA: no longer JP20.2
Other:
- note added: "0.45"
- note added: "SERVO CONNECTORS"
- note added: "UGV Simple Motherboard"
- note removed: "0.5"
- note removed: "Data Bus Baseboard"
- note removed: "ENCODER INTERFACE"
- note removed: "OUTPUT"
- note removed: "RC TAKEOVER SWITCH"
- note removed: "RX INPUT"
- moved on the sheet: C2, JP1, JP10, JP11, JP12, JP13, JP14, JP17, JP2, JP3, JP5, JP6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
