File: Electronics/Ranger I2C.sch (EAGLE design)
At the start: 22 parts, among them IC1 ATmega328P, J1 PWR, J2 I2C, J3 FTDI, J4 AN, J5 5V, J6 GND, J7 PWR, J8 PWR, Q1 16MHz

Commit message: Moved RC Mux to subdirectory. Minor changes to various other boards.
Parts:
- added C5: 470uF, rcl:CPOL-USE2.5-6
- added C6: 10uF, rcl:CPOL-USE2.5-6
- added J9: CAM, pinhead-2:PINHD-1X04_2.54-S
- C1, C2, C3, C4: device rcl:C-US050-025X075 -> rcl:C-US050-024X044
Connections:
- net 5V: now also C5.+, C6.+, J9.1
- net <RXD/TXO: now also J9.2
- net GND: now also C5.-, C6.-, J9.4
- net LV_TXD/RXI>: now also J9.3
Other:
- moved on the sheet: C1, C2, LED2, R1, R5, R7, S1
