File: Electronics/Serial I2C Bridge Prop.sch (EAGLE design)
At the start: 25 parts, among them IC1 24LC256SN, Q1 5MHz

Commit message: Moved RC Mux to subdirectory. Minor changes to various other boards.
Parts:
- R1, R2, R3, R4, R5, R6: value 22K -> 1.8K
- R10, R9: value 330 -> 390
Changed lines of the file:
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@@
 <grid distance="0.1" unitdist="inch" unit="inch" style="lines" multiple="1" display="no" altdistance="0.01" altunitdist="inch" altunit="inch"/>
 <layers>
-<layer number="1" name="Top" color="4" fill="1" visible="yes" active="no"/>
-<layer number="16" name="Bottom" color="1" fill="1" visible="yes" active="no"/>
-<layer number="17" name="Pads" color="2" fill="1" visible="yes" active="no"/>
-<layer number="18" name="Vias" color="2" fill="1" visible="yes" active="no"/>
-<layer number="19" name="Unrouted" color="6" fill="1" visible="yes" active="no"/>
-<layer number="20" name="Dimension" color="15" fill="1" visible="yes" active="no"/>
-<layer number="21" name="tPlace" color="7" fill="1" visible="yes" active="no"/>
-<layer number="22" name="bPlace" color="7" fill="1" visible="yes" active="no"/>
-<layer number="23" name="tOrigins" color="15" fill="1" visible="yes" active="no"/>
-<layer number="24" name="bOrigins" color="15" fill="1" visible="yes" active="no"/>
-<layer number="25" name="tNames" color="7" fill="1" visible="yes" active="no"/>
-<layer number="26" name="bNames" color="7" fill="1" visible="yes" active="no"/>
-<layer number="27" name="tValues" color="7" fill="1" visible="yes" active="no"/>
-<layer number="28" name="bValues" color="7" fill="1" visible="yes" active="no"/>
+<layer number="1" name="Top" color="4" fill="1" visible="no" active="no"/>
+<layer number="16" name="Bottom" color="1" fill="1" visible="no" active="no"/>
+<layer number="17" name="Pads" color="2" fill="1" visible="no" active="no"/>
+<layer number="18" name="Vias" color="2" fill="1" visible="no" active="no"/>
+<layer number="19" name="Unrouted" color="6" fill="1" visible="no" active="no"/>
+<layer number="20" name="Dimension" color="15" fill="1" visible="no" active="no"/>
+<layer number="21" name="tPlace" color="7" fill="1" visible="no" active="no"/>
+<layer number="22" name="bPlace" color="7" fill="1" visible="no" active="no"/>
+<layer number="23" name="tOrigins" color="15" fill="1" visible="no" active="no"/>
+<layer number="24" name="bOrigins" color="15" fill="1" visible="no" active="no"/>
+<layer number="25" name="tNames" color="7" fill="1" visible="no" active="no"/>
+<layer number="26" name="bNames" color="7" fill="1" visible="no" active="no"/>
+<layer number="27" name="tValues" color="7" fill="1" visible="no" active="no"/>
+<layer number="28" name="bValues" color="7" fill="1" visible="no" active="no"/>
 <layer number="29" name="tStop" color="7" fill="3" visible="no" active="no"/>
 <layer number="30" name="bStop" color="7" fill="6" visible="no" active="no"/>
@@
 <layer number="35" name="tGlue" color="7" fill="4" visible="no" active="no"/>
 <layer number="36" name="bGlue" color="7" fill="5" visible="no" active="no"/>
-<layer number="37" name="tTest" color="7" fill="1" visible="yes" active="no"/>
-<layer number="38" name="bTest" color="7" fill="1" visible="yes" active="no"/>
+<layer number="37" name="tTest" color="7" fill="1" visible="no" active="no"/>
+<layer number="38" name="bTest" color="7" fill="1" visible="no" active="no"/>
 <layer number="39" name="tKeepout" color="4" fill="11" visible="no" active="no"/>
 <layer number="40" name="bKeepout" color="1" fill="11" visible="no" active="no"/>
@@
 <layer number="44" name="Drills" color="7" fill="1" visible="no" active="no"/>
 <layer number="45" name="Holes" color="7" fill="1" visible="no" active="no"/>
-<layer number="46" name="Milling" color="3" fill="1" visible="yes" active="no"/>
-<layer number="47" name="Measures" color="7" fill="1" visible="yes" active="no"/>
-<layer number="48" name="Document" color="7" fill="1" visible="yes" active="no"/>
-<layer number="49" name="Reference" color="7" fill="1" visible="yes" active="no"/>
-<layer number="50" name="dxf" color="7" fill="1" visible="yes" active="no"/>
-<layer number="51" name="tDocu" color="7" fill="1" visible="yes" active="no"/>
-<layer number="52" name="bDocu" color="7" fill="1" visible="yes" active="no"/>
-<layer number="53" name="tPadExt" color="7" fill="1" visible="yes" active="no"/>
-<layer number="54" name="bPadExt" color="1" fill="1" visible="yes" active="no"/>
-<layer number="56" name="wert" color="7" fill="1" visible="yes" active="no"/>
+<layer number="46" name="Milling" color="3" fill="1" visible="no" active="no"/>
+<layer number="47" name="Measures" color="7" fill="1" visible="no" active="no"/>
+<layer number="48" name="Document" color="7" fill="1" visible="no" active="no"/>
+<layer number="49" name="Reference" color="7" fill="1" visible="no" active="no"/>
+<layer number="50" name="dxf" color="7" fill="1" visible="no" active="no"/>
+<layer number="51" name="tDocu" color="7" fill="1" visible="no" active="no"/>
+<layer number="52" name="bDocu" color="7" fill="1" visible="no" active="no"/>
+<layer number="53" name="tPadExt" color="7" fill="1" visible="no" active="no"/>
+<layer number="54" name="bPadExt" color="1" fill="1" visible="no" active="no"/>
+<layer number="56" name="wert" color="7" fill="1" visible="no" active="no"/>
 <layer number="91" name="Nets" color="2" fill="1" visible="yes" active="yes"/>
 <layer number="92" name="Busses" color="1" fill="1" visible="yes" active="yes"/>
@@
 <part name="JP5" library="pinhead-2" deviceset="PINHD-1X04" device="_2.54" value="DIAG"/>
 <part name="D1" library="diode" deviceset="1N4148" device="DO35-7" value="1N4148"/>
-<part name="R1" library="rcl" deviceset="R-US_" device="0204/5" value="22K"/>
-<part name="R2" library="rcl" deviceset="R-US_" device="0204/5" value="22K"/>
-<part name="R3" library="rcl" deviceset="R-US_" device="0204/5" value="22K"/>
-<part name="R4" library="rcl" deviceset="R-US_" device="0204/5" value="22K"/>
+<part name="R1" library="rcl" deviceset="R-US_" device="0204/5" value="1.8K"/>
+<part name="R2" library="rcl" deviceset="R-US_" device="0204/5" value="1.8K"/>
+<part name="R3" library="rcl" deviceset="R-US_" device="0204/5" value="1.8K"/>
+<part name="R4" library="rcl" deviceset="R-US_" device="0204/5" value="1.8K"/>
 <part name="U$4" library="parallax_propeller" deviceset="P8X32A-Q44" device=""/>
 <part name="C1" library="rcl" deviceset="C-US" device="C0603"/>
@@
 <part name="S1" library="mes_electromech" deviceset="SPST" device="TACTILE2" value="RESET"/>
 <part name="JP1" library="pinhead-2" deviceset="PINHD-1X06" device="_2.54" value="FTDI"/>
-<part name="R6" library="rcl" deviceset="R-US_" device="0204/5" value="22K"/>
+<part name="R6" library="rcl" deviceset="R-US_" device="0204/5" value="1.8K"/>
 <part name="D2" library="diode" deviceset="1N4148" device="DO35-7" value="1N4148"/>
-<part name="R5" library="rcl" deviceset="R-US_" device="0204/5" value="22K"/>
+<part name="R5" library="rcl" deviceset="R-US_" device="0204/5" value="1.8K"/>
 <part name="IC1" library="microchip" deviceset="24*" device="SN" technology="LC256"/>
 <part name="R7" library="rcl" deviceset="R-US_" device="0204/5" value="10K"/>
@@
 <part name="D3" library="special" deviceset="DUOLED" device=""/>
 <part name="GND5" library="mes" deviceset="GND" device=""/>
-<part name="R9" library="rcl" deviceset="R-US_" device="0204/5" value="330"/>
-<part name="R10" library="rcl" deviceset="R-US_" device="0204/5" value="330"/>
+<part name="R9" library="rcl" deviceset="R-US_" device="0204/5" value="390"/>
+<part name="R10" library="rcl" deviceset="R-US_" device="0204/5" value="390"/>
 </parts>
 <sheets>
