File: RoverMux/electronics/RC_MUX.sch (EAGLE design)
At the start: 24 parts, among them U1 TINY13, U2 MCP1824T, U3 74LS157D

Commit message: Consolidated RoverMux electronics and software directories under a single top-level directory
Parts:
- removed JP2: RESET, pinhead-2:PINHD-1X01_2.54-S
- added J1: ISP, bt_avr:AVRISP6
Connections:
- removed net LEDS: LED1.C, LED2.A, R2.1
- removed net N$1: SJ1.1, U1.(MOSI)PB0
- new net A: LED1.A, U1.(ADC2)PB4
- new net MISO: J1.MISO
- new net MOSI: J1.MOSI, SJ1.1, U1.(MOSI)PB0
- new net N$3: LED1.C, LED2.C, R2.1
- net !RESET: now also J1.!RESET; no longer JP2.1
- net +5V: now also J1.VCC; no longer LED1.A
- net B: now also LED2.A, U1.(ADC3)PB3; no longer R2.2, U1.(ADC2)PB4
- net CH1RX: now also J1.SCK
- net GND: now also J1.GND, R2.2; no longer LED2.C
Other:
- note added: "0.3"
- note removed: "0.2"
- note removed: "Want to flash the Tiny13? Use an 8SOIC clip or, MOSI=CH3RX, (connect jumper) MISO=CH2RX, SCK=CH1RX, power with VCC/GND and connect programmer's VTG to VCC and GND to GND, and use exposed RESET pin"
- moved on the sheet: LED1, LED2, R2
Changed lines of the file:
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@@
 </part>
 <part name="GND4" library="mes" deviceset="GND" device=""/>
-<part name="SUPPLY6" library="supply2" deviceset="+5V" device=""/>
 <part name="U2" library="mes_regulators" deviceset="MCP1801" device="" value="MCP1824T">
 <attribute name="PARTNO" value="MCP1824T-5002E/OT"/>
@@
 </part>
 <part name="SJ1" library="SparkFun" deviceset="SOLDERJUMPER" device="NC2" value="CH3"/>
-<part name="JP2" library="pinhead-2" deviceset="PINHD-1X01" device="_2.54-S" value="RESET"/>
+<part name="J1" library="bt_avr" deviceset="AVRISP6" device="" value="ISP"/>
+<part name="SUPPLY6" library="supply2" deviceset="+5V" device=""/>
+<part name="GND3" library="mes" deviceset="GND" device=""/>
 </parts>
 <sheets>
@@
 <plain>
 <text x="162.56" y="22.86" size="3.81" layer="94">RC MUX</text>
-<text x="233.68" y="22.86" size="3.81" layer="94">0.2</text>
-<text x="91.44" y="40.64" size="1.778" layer="91">Want to flash the Tiny13?
-Use an 8SOIC clip or,
-MOSI=CH3RX, (connect jumper)
-MISO=CH2RX,
-SCK=CH1RX,
-power with VCC/GND and
-connect programmer's VTG to VCC and
-GND to GND,
-and use exposed RESET pin</text>
+<text x="233.68" y="22.86" size="3.81" layer="94">0.3</text>
 </plain>
 <instances>
@@
 <attribute name="PARTNO" x="22.86" y="121.92" size="1.778" layer="96" display="off"/>
 </instance>
-<instance part="R2" gate="G$1" x="104.14" y="129.54" rot="R180">
-<attribute name="PARTNO" x="104.14" y="129.54" size="1.778" layer="96" rot="R270" display="off"/>
+<instance part="R2" gate="G$1" x="116.84" y="96.52" rot="R270">
+<attribute name="PARTNO" x="116.84" y="96.52" size="1.778" layer="96" display="off"/>
 </instance>
 <instance part="SUPPLY1" gate="G$1" x="144.78" y="167.64"/>
@@
 <instance part="SUPPLY4" gate="+5V" x="83.82" y="165.1"/>
 <instance part="GND1" gate="1" x="33.02" y="101.6"/>
-<instance part="GND2" gate="1" x="111.76" y="106.68"/>
+<instance part="GND2" gate="1" x="116.84" y="86.36"/>
 <instance part="GND5" gate="1" x="220.98" y="81.28"/>
 <instance part="GND6" gate="1" x="142.24" y="66.04"/>
 <instance part="SUPPLY7" gate="G$1" x="218.44" y="137.16"/>
 <instance part="GND7" gate="1" x="165.1" y="73.66"/>
-<instance part="LED1" gate="G$1" x="111.76" y="139.7">
-<attribute name="PARTNO" x="111.76" y="139.7" size="1.778" layer="96" display="off"/>
-</instance>
-<instance part="LED2" gate="G$1" x="111.76" y="121.92">
-<attribute name="PARTNO" x="111.76" y="121.92" size="1.778" layer="96" display="off"/>
+<instance part="LED1" gate="G$1" x="121.92" y="111.76">
+<attribute name="PARTNO" x="121.92" y="111.76" size="1.778" layer="96" display="off"/>
+</instance>
+<instance part="LED2" gate="G$1" x="111.76" y="111.76">
+<attribute name="PARTNO" x="111.76" y="111.76" size="1.778" layer="96" display="off"/>
 </instance>
 <instance part="C4" gate="G$1" x="33.02" y="121.92">
@@
 </instance>
 <instance part="GND4" gate="1" x="25.4" y="50.8"/>
-<instance part="SUPPLY6" gate="+5V" x="111.76" y="149.86"/>
 <instance part="U2" gate="G$1" x="43.18" y="73.66" rot="MR0">
 <attribute name="PARTNO" x="43.18" y="73.66" size="1.778" layer="96" rot="MR0" display="off"/>
@@
 </instance>
 <instance part="SJ1" gate="1" x="88.9" y="119.38" smashed="yes"/>
-<instance part="JP2" gate="A" x="99.06" y="144.78"/>
+<instance part="J1" gate="A" x="48.26" y="17.78"/>
+<instance part="SUPPLY6" gate="+5V" x="30.48" y="30.48"/>
+<instance part="GND3" gate="1" x="30.48" y="17.78"/>
 </instances>
 <busses>
@@
 <net name="!RESET" class="0">
 <segment>
-<wire x1="83.82" y1="132.08" x2="83.82" y2="144.78" width="0.1524" layer="91"/>
+<wire x1="83.82" y1="132.08" x2="83.82" y2="149.86" width="0.1524" layer="91"/>
 <pinref part="R1" gate="G$1" pin="1"/>
 <pinref part="U1" gate="G$1" pin="(RESET)PB5"/>
-<wire x1="83.82" y1="144.78" x2="83.82" y2="149.86" width="0.1524" layer="91"/>
 <wire x1="81.28" y1="132.08" x2="83.82" y2="132.08" width="0.1524" layer="91"/>
-<pinref part="JP2" gate="A" pin="1"/>
-<wire x1="96.52" y1="144.78" x2="83.82" y2="144.78" width="0.1524" layer="91"/>
-<junction x="83.82" y="144.78"/>
+</segment>
+<segment>
+<pinref part="J1" gate="A" pin="!RESET"/>
+<wire x1="63.5" y1="25.4" x2="76.2" y2="25.4" width="0.1524" layer="91"/>
+<label x="76.2" y="25.4" size="1.778" layer="95" rot="MR0"/>
 </segment>
 </net>
@@
 <wire x1="81.28" y1="124.46" x2="104.14" y2="124.46" width="0.1524" layer="91"/>
 <label x="104.14" y="124.46" size="1.778" layer="95" rot="MR0"/>
+</segment>
+<segment>
+<pinref part="J1" gate="A" pin="SCK"/>
+<wire x1="63.5" y1="22.86" x2="76.2" y2="22.86" width="0.1524" layer="91"/>
+<label x="76.2" y="22.86" size="1.778" layer="95" rot="MR0"/>
 </segment>
 </net>
@@
 </segment>
 <segment>
-<pinref part="LED2" gate="G$1" pin="C"/>
-<wire x1="111.76" y1="109.22" x2="111.76" y2="116.84" width="0.1524" layer="91"/>
 <pinref part="GND2" gate="1" pin="GND"/>
+<pinref part="R2" gate="G$1" pin="2"/>
+<wire x1="116.84" y1="91.44" x2="116.84" y2="88.9" width="0.1524" layer="91"/>
+</segment>
+<segment>
+<pinref part="J1" gate="A" pin="GND"/>
+<wire x1="33.02" y1="22.86" x2="30.48" y2="22.86" width="0.1524" layer="91"/>
+<wire x1="30.48" y1="22.86" x2="30.48" y2="20.32" width="0.1524" layer="91"/>
+<pinref part="GND3" gate="1" pin="GND"/>
 </segment>
 </net>
@@
 </segment>
 <segment>
+<pinref part="J1" gate="A" pin="VCC"/>
+<wire x1="33.02" y1="25.4" x2="30.48" y2="25.4" width="0.1524" layer="91"/>
+<wire x1="30.48" y1="25.4" x2="30.48" y2="27.94" width="0.1524" layer="91"/>
 <pinref part="SUPPLY6" gate="+5V" pin="+5V"/>
-<wire x1="111.76" y1="147.32" x2="111.76" y2="142.24" width="0.1524" layer="91"/>
-<pinref part="LED1" gate="G$1" pin="A"/>
 </segment>
 </net>
@@
 </segment>
 <segment>
-<pinref part="R2" gate="G$1" pin="2"/>
-<pinref part="U1" gate="G$1" pin="(ADC2)PB4"/>
-<wire x1="81.28" y1="129.54" x2="99.06" y2="129.54" width="0.1524" layer="91"/>
-<label x="93.98" y="129.54" size="1.778" layer="95"/>
-</segment>
-</net>
-<net name="LEDS" class="0">
-<segment>
-<wire x1="109.22" y1="129.54" x2="111.76" y2="129.54" width="0.1524" layer="91"/>
-<wire x1="111.76" y1="129.54" x2="111.76" y2="134.62" width="0.1524" layer="91"/>
-<pinref part="R2" gate="G$1" pin="1"/>
-<pinref part="LED1" gate="G$1" pin="C"/>
 <pinref part="LED2" gate="G$1" pin="A"/>
-<wire x1="111.76" y1="129.54" x2="111.76" y2="124.46" width="0.1524" layer="91"/>
-<junction x="111.76" y="129.54"/>
-</segment>
-</net>
-<net name="N$1" class="0">
+<wire x1="111.76" y1="127" x2="111.76" y2="114.3" width="0.1524" layer="91"/>
+<pinref part="U1" gate="G$1" pin="(ADC3)PB3"/>
+<wire x1="111.76" y1="127" x2="81.28" y2="127" width="0.1524" layer="91"/>
+<label x="104.14" y="127" size="1.778" layer="95" rot="MR0"/>
+</segment>
+</net>
+<net name="MOSI" class="0">
 <segment>
 <pinref part="U1" gate="G$1" pin="(MOSI)PB0"/>
 <pinref part="SJ1" gate="1" pin="1"/>
 <wire x1="83.82" y1="119.38" x2="81.28" y2="119.38" width="0.1524" layer="91"/>
+</segment>
+<segment>
+<pinref part="J1" gate="A" pin="MOSI"/>
+<wire x1="63.5" y1="20.32" x2="76.2" y2="20.32" width="0.1524" layer="91"/>
+<label x="76.2" y="20.32" size="1.778" layer="95" rot="MR0"/>
+</segment>
+</net>
+<net name="A" class="0">
+<segment>
+<wire x1="121.92" y1="129.54" x2="121.92" y2="114.3" width="0.1524" layer="91"/>
+<pinref part="LED1" gate="G$1" pin="A"/>
+<pinref part="U1" gate="G$1" pin="(ADC2)PB4"/>
+<wire x1="121.92" y1="129.54" x2="81.28" y2="129.54" width="0.1524" layer="91"/>
+<label x="104.14" y="129.54" size="1.778" layer="95" rot="MR0"/>
+</segment>
+</net>
+<net name="N$3" class="0">
+<segment>
+<pinref part="LED2" gate="G$1" pin="C"/>
+<wire x1="111.76" y1="106.68" x2="111.76" y2="104.14" width="0.1524" layer="91"/>
+<pinref part="LED1" gate="G$1" pin="C"/>
+<wire x1="111.76" y1="104.14" x2="116.84" y2="104.14" width="0.1524" layer="91"/>
+<wire x1="116.84" y1="104.14" x2="121.92" y2="104.14" width="0.1524" layer="91"/>
+<wire x1="121.92" y1="104.14" x2="121.92" y2="106.68" width="0.1524" layer="91"/>
+<pinref part="R2" gate="G$1" pin="1"/>
+<wire x1="116.84" y1="101.6" x2="116.84" y2="104.14" width="0.1524" layer="91"/>
+<junction x="116.84" y="104.14"/>
+</segment>
+</net>
+<net name="MISO" class="0">
+<segment>
+<pinref part="J1" gate="A" pin="MISO"/>
+<wire x1="63.5" y1="17.78" x2="76.2" y2="17.78" width="0.1524" layer="91"/>
+<label x="76.2" y="17.78" size="1.778" layer="95" rot="MR0"/>
 </segment>
 </net>
@@
 </schematic>
 </drawing>
-<compatibility>
-<note version="6.3" minversion="6.2.2" severity="warning">
-Since Version 6.2.2 text objects can contain more than one line,
-which will not be processed correctly with this version.
-</note>
-</compatibility>
 </eagle>
