File: RoverMeter/electronics/RoverMeter.sch (EAGLE design)
At the start: 17 parts, among them IC1 INA168, IC3 TINY85, J1 AVRISP, U1 MCP1824

Commit message: Revised board layout somewhat
Parts:
- removed U1: MCP1824, bt_regulator:MCP1824
- added IC2: KA78L05AIMTF, v-reg-3:78LXX-SOT89
- R1: device rcl:R-US_R4527 -> bt:R-US_WSLP3921; PARTNO (none) -> WSLP3921L5000FEB; POWER (none) -> 6W+
Connections:
- net 5V: now also IC2.OUT; no longer U1.OUT
- net GND: now also IC2.GND; no longer U1.GND
- net V+: now also IC2.IN; no longer U1.EN, U1.IN
Other:
- note removed: "Verify Regulator input voltage"
Changed lines of the file:
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@@
 </classes>
 <parts>
-<part name="R1" library="rcl" deviceset="R-US_" device="R4527" value="0.001"/>
+<part name="R1" library="bt" deviceset="R-US_" device="WSLP3921" value="0.001">
+<attribute name="PARTNO" value="WSLP3921L5000FEB"/>
+<attribute name="POWER" value="6W+"/>
+</part>
 <part name="IC1" library="burr-brown" deviceset="INA168" device=""/>
 <part name="GND1" library="SparkFun" deviceset="GND" device=""/>
@@
 <part name="U$2" library="bt" deviceset="5V" device=""/>
 <part name="GND2" library="bt" deviceset="GND" device=""/>
-<part name="U1" library="bt_regulator" deviceset="MCP1824" device=""/>
 <part name="SUPPLY3" library="supply2" deviceset="V+" device=""/>
 <part name="IC3" library="bt_avr" deviceset="TINY25/45/85" device="-20SU" value="TINY85"/>
@@
 <part name="U$1" library="bt" deviceset="5V" device=""/>
 <part name="R5" library="resistor" deviceset="R-US_" device="R0603" value="10K"/>
+<part name="IC2" library="v-reg-3" deviceset="78LXX" device="-SOT89" value="KA78L05AIMTF">
+<attribute name="VOLTAGE" value="30V"/>
+</part>
 </parts>
 <sheets>
@@
 <text x="35.56" y="22.86" size="1.778" layer="94">Verify design for:
 2S-3S (12.6V), 150A ideally</text>
-<text x="50.8" y="152.4" size="1.778" layer="91">Verify Regulator input voltage</text>
 </plain>
 <instances>
-<instance part="R1" gate="G$1" x="78.74" y="101.6"/>
+<instance part="R1" gate="G$1" x="78.74" y="101.6">
+<attribute name="POWER" x="76.454" y="95.758" size="1.778" layer="96"/>
+<attribute name="PARTNO" x="75.184" y="93.218" size="1.778" layer="96"/>
+</instance>
 <instance part="IC1" gate="G$1" x="101.6" y="71.12"/>
 <instance part="GND1" gate="1" x="116.84" y="40.64"/>
@@
 <instance part="U$2" gate="G$1" x="83.82" y="154.94"/>
 <instance part="GND2" gate="1" x="27.94" y="119.38"/>
-<instance part="U1" gate="G$1" x="55.88" y="142.24"/>
-<instance part="SUPPLY3" gate="1" x="43.18" y="157.48"/>
+<instance part="SUPPLY3" gate="1" x="27.94" y="157.48"/>
 <instance part="IC3" gate="1" x="187.96" y="139.7" rot="MR0"/>
 <instance part="U$3" gate="G$1" x="226.06" y="154.94"/>
@@
 <instance part="U$1" gate="G$1" x="147.32" y="167.64"/>
 <instance part="R5" gate="G$1" x="147.32" y="157.48" rot="R90"/>
+<instance part="IC2" gate="1" x="43.18" y="147.32">
+<attribute name="VOLTAGE" x="45.72" y="134.62" size="1.778" layer="96"/>
+</instance>
 </instances>
 <busses>
@@
 <wire x1="68.58" y1="127" x2="83.82" y2="127" width="0.1524" layer="91"/>
 <wire x1="83.82" y1="127" x2="83.82" y2="144.78" width="0.1524" layer="91"/>
-<pinref part="U1" gate="G$1" pin="GND"/>
-<wire x1="45.72" y1="142.24" x2="40.64" y2="142.24" width="0.1524" layer="91"/>
-<wire x1="40.64" y1="142.24" x2="40.64" y2="127" width="0.1524" layer="91"/>
 <pinref part="GND2" gate="1" pin="GND"/>
 <pinref part="C4" gate="G$1" pin="2"/>
-<junction x="40.64" y="127"/>
-<wire x1="68.58" y1="127" x2="40.64" y2="127" width="0.1524" layer="91"/>
-<wire x1="40.64" y1="127" x2="27.94" y2="127" width="0.1524" layer="91"/>
+<wire x1="68.58" y1="127" x2="43.18" y2="127" width="0.1524" layer="91"/>
+<wire x1="43.18" y1="127" x2="27.94" y2="127" width="0.1524" layer="91"/>
 <wire x1="27.94" y1="121.92" x2="27.94" y2="127" width="0.1524" layer="91"/>
 <junction x="27.94" y="127"/>
 <wire x1="27.94" y1="127" x2="27.94" y2="134.62" width="0.1524" layer="91"/>
 <junction x="68.58" y="127"/>
+<pinref part="IC2" gate="1" pin="GND"/>
+<wire x1="43.18" y1="139.7" x2="43.18" y2="127" width="0.1524" layer="91"/>
+<junction x="43.18" y="127"/>
 </segment>
 <segment>
@@
 </segment>
 <segment>
-<pinref part="U1" gate="G$1" pin="IN"/>
 <pinref part="SUPPLY3" gate="1" pin="V+"/>
-<wire x1="45.72" y1="147.32" x2="43.18" y2="147.32" width="0.1524" layer="91"/>
-<wire x1="43.18" y1="147.32" x2="43.18" y2="154.94" width="0.1524" layer="91"/>
-<pinref part="U1" gate="G$1" pin="EN"/>
-<wire x1="45.72" y1="137.16" x2="43.18" y2="137.16" width="0.1524" layer="91"/>
-<wire x1="43.18" y1="137.16" x2="43.18" y2="147.32" width="0.1524" layer="91"/>
-<junction x="43.18" y="147.32"/>
+<wire x1="35.56" y1="147.32" x2="27.94" y2="147.32" width="0.1524" layer="91"/>
+<wire x1="27.94" y1="147.32" x2="27.94" y2="154.94" width="0.1524" layer="91"/>
+<junction x="27.94" y="147.32"/>
 <pinref part="C4" gate="G$1" pin="1"/>
-<wire x1="43.18" y1="147.32" x2="27.94" y2="147.32" width="0.1524" layer="91"/>
 <wire x1="27.94" y1="147.32" x2="27.94" y2="142.24" width="0.1524" layer="91"/>
+<pinref part="IC2" gate="1" pin="IN"/>
 </segment>
 </net>
@@
 <net name="5V" class="0">
 <segment>
-<pinref part="U1" gate="G$1" pin="OUT"/>
 <pinref part="U$2" gate="G$1" pin="5V"/>
-<wire x1="63.5" y1="147.32" x2="68.58" y2="147.32" width="0.1524" layer="91"/>
+<wire x1="50.8" y1="147.32" x2="68.58" y2="147.32" width="0.1524" layer="91"/>
 <wire x1="68.58" y1="147.32" x2="83.82" y2="147.32" width="0.1524" layer="91"/>
 <wire x1="83.82" y1="147.32" x2="83.82" y2="152.4" width="0.1524" layer="91"/>
@@
 <pinref part="C3" gate="G$1" pin="1"/>
 <wire x1="68.58" y1="142.24" x2="68.58" y2="147.32" width="0.1524" layer="91"/>
-</segment>
-<segment>
+<pinref part="IC2" gate="1" pin="OUT"/>
+<junction x="68.58" y="147.32"/>
+<label x="53.34" y="147.32" size="1.778" layer="95"/>
+</segment>
+<segment>
