File: RoverBaseboard/Motherboard_lpcxpresso.sch (EAGLE design)
At the start: 60 parts, among them IC1 7805, IC3 3.3V, U2 microSD

Commit message: Minor modifications
Other:
- note removed: "3v3 regulator required?"
- note removed: "CAN pins can be used as GPIO, interrupts (encoders)"
- note removed: "I2C & UART layout works"
- note removed: "I2C/Serial/SPI peripherals are NOT allocated twice?"
Changed lines of the file:
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@@
 <text x="174.752" y="142.494" size="1.778" layer="97" rot="MR0">MBED</text>
 <text x="152.4" y="238.76" size="2.54" layer="91">Verify:</text>
-<text x="154.94" y="233.68" size="2.54" layer="91">I2C &amp; UART layout works</text>
 <text x="154.94" y="228.6" size="2.54" layer="91">ISP bootloader can work w/ zigbee</text>
 <text x="152.4" y="243.84" size="2.54" layer="91">Add Capacitors</text>
-<text x="154.94" y="223.52" size="2.54" layer="91">CAN pins can be used as GPIO, interrupts (encoders)</text>
 <text x="14.732" y="142.24" size="1.778" layer="97">MBED</text>
 <wire x1="0" y1="248.92" x2="480.06" y2="248.92" width="0.1524" layer="94"/>
@@
 <text x="76.2" y="208.28" size="2.54" layer="97">LPXpresso / MBED</text>
 <text x="322.58" y="76.2" size="1.778" layer="97">POWER SUPPLY</text>
-<text x="154.94" y="213.36" size="2.54" layer="91">3v3 regulator required?</text>
-<text x="154.94" y="218.44" size="2.54" layer="91">I2C/Serial/SPI peripherals are NOT allocated twice?</text>
 </plain>
 <instances>
