File: RoverBaseboard/RoverBaseboard.sch (EAGLE design)
At the start: 58 parts, among them IC1 7805, IC3 3.3V, U2 microSD

Commit message: Bugfix to supply--3.3V regulator now feeds LPCXpresso. Minor tweaks. Powering analog ports more directly. Rerouted power. Moved power pins to align to 0.1" spacing. Heat sink now connected to 3V3 out.
Connections:
- removed net SINK: IC3.OUT@1
- net +3V3: now also IC3.OUT@1, U$1.VOUT/3.3V
- net +5V: no longer U$1.EXT_POWX
Changed lines of the file:
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@@
 <grid distance="0.1" unitdist="inch" unit="inch" style="lines" multiple="1" display="no" altdistance="0.01" altunitdist="inch" altunit="inch"/>
 <layers>
-<layer number="1" name="Top" color="4" fill="1" visible="yes" active="no"/>
-<layer number="16" name="Bottom" color="1" fill="1" visible="yes" active="no"/>
-<layer number="17" name="Pads" color="2" fill="1" visible="yes" active="no"/>
-<layer number="18" name="Vias" color="2" fill="1" visible="yes" active="no"/>
-<layer number="19" name="Unrouted" color="6" fill="1" visible="yes" active="no"/>
-<layer number="20" name="Dimension" color="15" fill="1" visible="yes" active="no"/>
-<layer number="21" name="tPlace" color="7" fill="1" visible="yes" active="no"/>
-<layer number="22" name="bPlace" color="7" fill="1" visible="yes" active="no"/>
-<layer number="23" name="tOrigins" color="15" fill="1" visible="yes" active="no"/>
-<layer number="24" name="bOrigins" color="15" fill="1" visible="yes" active="no"/>
-<layer number="25" name="tNames" color="7" fill="1" visible="yes" active="no"/>
-<layer number="26" name="bNames" color="7" fill="1" visible="yes" active="no"/>
-<layer number="27" name="tValues" color="7" fill="1" visible="yes" active="no"/>
-<layer number="28" name="bValues" color="7" fill="1" visible="yes" active="no"/>
+<layer number="1" name="Top" color="4" fill="1" visible="no" active="no"/>
+<layer number="16" name="Bottom" color="1" fill="1" visible="no" active="no"/>
+<layer number="17" name="Pads" color="2" fill="1" visible="no" active="no"/>
+<layer number="18" name="Vias" color="2" fill="1" visible="no" active="no"/>
+<layer number="19" name="Unrouted" color="6" fill="1" visible="no" active="no"/>
+<layer number="20" name="Dimension" color="15" fill="1" visible="no" active="no"/>
+<layer number="21" name="tPlace" color="7" fill="1" visible="no" active="no"/>
+<layer number="22" name="bPlace" color="7" fill="1" visible="no" active="no"/>
+<layer number="23" name="tOrigins" color="15" fill="1" visible="no" active="no"/>
+<layer number="24" name="bOrigins" color="15" fill="1" visible="no" active="no"/>
+<layer number="25" name="tNames" color="7" fill="1" visible="no" active="no"/>
+<layer number="26" name="bNames" color="7" fill="1" visible="no" active="no"/>
+<layer number="27" name="tValues" color="7" fill="1" visible="no" active="no"/>
+<layer number="28" name="bValues" color="7" fill="1" visible="no" active="no"/>
 <layer number="29" name="tStop" color="7" fill="3" visible="no" active="no"/>
 <layer number="30" name="bStop" color="7" fill="6" visible="no" active="no"/>
@@
 <layer number="35" name="tGlue" color="7" fill="4" visible="no" active="no"/>
 <layer number="36" name="bGlue" color="7" fill="5" visible="no" active="no"/>
-<layer number="37" name="tTest" color="7" fill="1" visible="yes" active="no"/>
-<layer number="38" name="bTest" color="7" fill="1" visible="yes" active="no"/>
+<layer number="37" name="tTest" color="7" fill="1" visible="no" active="no"/>
+<layer number="38" name="bTest" color="7" fill="1" visible="no" active="no"/>
 <layer number="39" name="tKeepout" color="4" fill="11" visible="no" active="no"/>
 <layer number="40" name="bKeepout" color="1" fill="11" visible="no" active="no"/>
@@
 <layer number="44" name="Drills" color="7" fill="1" visible="no" active="no"/>
 <layer number="45" name="Holes" color="7" fill="1" visible="no" active="no"/>
-<layer number="46" name="Milling" color="3" fill="1" visible="yes" active="no"/>
-<layer number="47" name="Measures" color="7" fill="1" visible="yes" active="no"/>
-<layer number="48" name="Document" color="7" fill="1" visible="yes" active="no"/>
-<layer number="49" name="Reference" color="7" fill="1" visible="yes" active="no"/>
-<layer number="50" name="dxf" color="7" fill="1" visible="yes" active="no"/>
-<layer number="51" name="tDocu" color="7" fill="1" visible="yes" active="no"/>
-<layer number="52" name="bDocu" color="7" fill="1" visible="yes" active="no"/>
-<layer number="53" name="tGND_GNDA" color="7" fill="9" visible="yes" active="no"/>
-<layer number="54" name="bGND_GNDA" color="1" fill="9" visible="yes" active="no"/>
-<layer number="56" name="wert" color="7" fill="1" visible="yes" active="no"/>
+<layer number="46" name="Milling" color="3" fill="1" visible="no" active="no"/>
+<layer number="47" name="Measures" color="7" fill="1" visible="no" active="no"/>
+<layer number="48" name="Document" color="7" fill="1" visible="no" active="no"/>
+<layer number="49" name="Reference" color="7" fill="1" visible="no" active="no"/>
+<layer number="50" name="dxf" color="7" fill="1" visible="no" active="no"/>
+<layer number="51" name="tDocu" color="7" fill="1" visible="no" active="no"/>
+<layer number="52" name="bDocu" color="7" fill="1" visible="no" active="no"/>
+<layer number="53" name="tGND_GNDA" color="7" fill="9" visible="no" active="no"/>
+<layer number="54" name="bGND_GNDA" color="1" fill="9" visible="no" active="no"/>
+<layer number="56" name="wert" color="7" fill="1" visible="no" active="no"/>
 <layer number="91" name="Nets" color="2" fill="1" visible="yes" active="yes"/>
 <layer number="92" name="Busses" color="1" fill="1" visible="yes" active="yes"/>
@@
 <part name="SUPPLY3" library="supply2" deviceset="GND" device=""/>
 <part name="SUPPLY4" library="supply2" deviceset="GND" device=""/>
-<part name="P+2" library="supply1" deviceset="+5V" device=""/>
 <part name="R5" library="rcl" deviceset="R-US_" device="R0603" value="2.2K">
 <attribute name="MF" value=""/>
@@
 <part name="IC1" library="v-reg-3" deviceset="78XXS" device="" value="7805"/>
 <part name="BECSEL" library="pinhead-2" deviceset="PINHD-1X03" device="_2.54-S" value="5V | 6V"/>
+<part name="+3V2" library="supply1" deviceset="+3V3" device=""/>
 </parts>
 <sheets>
@@
 </plain>
 <instances>
-<instance part="SUPPLY3" gate="GND" x="43.18" y="198.12"/>
+<instance part="SUPPLY3" gate="GND" x="15.24" y="182.88"/>
 <instance part="SUPPLY4" gate="GND" x="373.38" y="91.44"/>
-<instance part="P+2" gate="1" x="33.02" y="205.74"/>
 <instance part="R5" gate="G$1" x="215.9" y="185.42" rot="R90">
 <attribute name="OC_NEWARK" x="215.9" y="185.42" size="1.778" layer="96" display="off"/>
@@
 <instance part="IC1" gate="1" x="276.86" y="68.58"/>
 <instance part="BECSEL" gate="A" x="297.18" y="78.74"/>
+<instance part="+3V2" gate="G$1" x="132.08" y="203.2"/>
 </instances>
 <busses>
@@
 <net name="GND" class="0">
 <segment>
-<wire x1="63.5" y1="190.5" x2="35.56" y2="190.5" width="0.1524" layer="91"/>
-<wire x1="35.56" y1="190.5" x2="35.56" y2="200.66" width="0.1524" layer="91"/>
-<wire x1="35.56" y1="200.66" x2="43.18" y2="200.66" width="0.1524" layer="91"/>
+<wire x1="63.5" y1="190.5" x2="15.24" y2="190.5" width="0.1524" layer="91"/>
+<wire x1="15.24" y1="190.5" x2="15.24" y2="185.42" width="0.1524" layer="91"/>
 <pinref part="SUPPLY3" gate="GND" pin="GND"/>
 <pinref part="U$1" gate="G$1" pin="GND1"/>
@@
 <net name="+5V" class="0">
 <segment>
-<wire x1="63.5" y1="187.96" x2="33.02" y2="187.96" width="0.1524" layer="91"/>
-<wire x1="33.02" y1="187.96" x2="33.02" y2="203.2" width="0.1524" layer="91"/>
-<pinref part="P+2" gate="1" pin="+5V"/>
-<pinref part="U$1" gate="G$1" pin="EXT_POWX"/>
-</segment>
-<segment>
 <pinref part="P+3" gate="1" pin="+5V"/>
 <wire x1="327.66" y1="53.34" x2="327.66" y2="58.42" width="0.1524" layer="91"/>
@@
 <segment>
 <pinref part="IC3" gate="G$1" pin="OUT"/>
-<wire x1="350.52" y1="58.42" x2="360.68" y2="58.42" width="0.1524" layer="91"/>
+<wire x1="350.52" y1="58.42" x2="355.6" y2="58.42" width="0.1524" layer="91"/>
+<wire x1="355.6" y1="58.42" x2="360.68" y2="58.42" width="0.1524" layer="91"/>
 <wire x1="360.68" y1="58.42" x2="360.68" y2="68.58" width="0.1524" layer="91"/>
 <pinref part="+3V8" gate="G$1" pin="+3V3"/>
@@
 <wire x1="360.68" y1="53.34" x2="360.68" y2="58.42" width="0.1524" layer="91"/>
 <junction x="360.68" y="58.42"/>
+<pinref part="IC3" gate="G$1" pin="OUT@1"/>
+<wire x1="350.52" y1="55.88" x2="355.6" y2="55.88" width="0.1524" layer="91"/>
+<wire x1="355.6" y1="55.88" x2="355.6" y2="58.42" width="0.1524" layer="91"/>
+<junction x="355.6" y="58.42"/>
+</segment>
+<segment>
+<pinref part="U$1" gate="G$1" pin="VOUT/3.3V"/>
+<wire x1="124.46" y1="190.5" x2="132.08" y2="190.5" width="0.1524" layer="91"/>
+<wire x1="132.08" y1="190.5" x2="132.08" y2="200.66" width="0.1524" layer="91"/>
+<pinref part="+3V2" gate="G$1" pin="+3V3"/>
 </segment>
 </net>
@@
 </segment>
 </net>
-<net name="SINK" class="0">
-<segment>
-<pinref part="IC3" gate="G$1" pin="OUT@1"/>
-<wire x1="350.52" y1="55.88" x2="355.6" y2="55.88" width="0.1524" layer="91"/>
-<label x="350.52" y="55.88" size="1.778" layer="95"/>
-</segment>
-</net>

Commit message: Change to LDO regulator, added port labels for digital, analog, encoders, change cap values.
Parts:
- removed IC1: 7805, v-reg-3:78XXS
- added C1: 106, rcl:C-USC1206
- added U1: LD29150DT50R, bt_regulator:LD29150DT
- C10, C11, C12, C13, C14, C15, C2, C3, C4, C6, C8, C9: value 10 -> 106
- C17: value 100 -> 33uF
- C5, C7: value 0.1 -> 104
Connections:
- net +5V: now also U1.VOUT; no longer IC1.OUT
- net GND: now also C1.2, U1.GND; no longer IC1.GND
- net N$3: now also C1.1, U1.VIN; no longer IC1.IN
Other:
- moved on the sheet: BECSEL, C2, JP3
Changed lines of the file:
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@@
 <attribute name="OC_NEWARK" value="unknown"/>
 </part>
-<part name="C2" library="rcl" deviceset="C-US" device="C1206" value="10"/>
-<part name="C4" library="rcl" deviceset="C-US" device="C0603" value="10"/>
-<part name="C5" library="rcl" deviceset="C-US" device="C0603" value="0.1"/>
-<part name="C6" library="rcl" deviceset="C-US" device="C0603" value="10"/>
-<part name="C7" library="rcl" deviceset="C-US" device="C0603" value="0.1"/>
-<part name="C8" library="rcl" deviceset="C-US" device="C0603" value="10"/>
-<part name="C9" library="rcl" deviceset="C-US" device="C0603" value="10"/>
-<part name="C10" library="rcl" deviceset="C-US" device="C0603" value="10"/>
-<part name="C11" library="rcl" deviceset="C-US" device="C0603" value="10"/>
-<part name="C12" library="rcl" deviceset="C-US" device="C0603" value="10"/>
-<part name="C13" library="rcl" deviceset="C-US" device="C0603" value="10"/>
-<part name="C14" library="rcl" deviceset="C-US" device="C0603" value="10"/>
-<part name="C15" library="rcl" deviceset="C-US" device="C0603" value="10"/>
+<part name="C2" library="rcl" deviceset="C-US" device="C1206" value="106"/>
+<part name="C4" library="rcl" deviceset="C-US" device="C0603" value="106"/>
+<part name="C5" library="rcl" deviceset="C-US" device="C0603" value="104"/>
+<part name="C6" library="rcl" deviceset="C-US" device="C0603" value="106"/>
+<part name="C7" library="rcl" deviceset="C-US" device="C0603" value="104"/>
+<part name="C8" library="rcl" deviceset="C-US" device="C0603" value="106"/>
+<part name="C9" library="rcl" deviceset="C-US" device="C0603" value="106"/>
+<part name="C10" library="rcl" deviceset="C-US" device="C0603" value="106"/>
+<part name="C11" library="rcl" deviceset="C-US" device="C0603" value="106"/>
+<part name="C12" library="rcl" deviceset="C-US" device="C0603" value="106"/>
+<part name="C13" library="rcl" deviceset="C-US" device="C0603" value="106"/>
+<part name="C14" library="rcl" deviceset="C-US" device="C0603" value="106"/>
+<part name="C15" library="rcl" deviceset="C-US" device="C0603" value="106"/>
 <part name="SUPPLY12" library="supply2" deviceset="GND" device=""/>
-<part name="C3" library="rcl" deviceset="C-US" device="C1206" value="10"/>
+<part name="C3" library="rcl" deviceset="C-US" device="C1206" value="106"/>
 <part name="P+4" library="supply1" deviceset="+5V" device=""/>
 <part name="IC3" library="SparkFun" deviceset="V_REG_LM1117" device="SOT223" value="3.3V"/>
 <part name="+3V8" library="supply1" deviceset="+3V3" device=""/>
-<part name="C17" library="rcl" deviceset="CPOL-US" device="140CLH-0810" value="100"/>
-<part name="IC1" library="v-reg-3" deviceset="78XXS" device="" value="7805"/>
+<part name="C17" library="rcl" deviceset="CPOL-US" device="140CLH-0810" value="33uF"/>
 <part name="BECSEL" library="pinhead-2" deviceset="PINHD-1X03" device="_2.54-S" value="5V | 6V"/>
 <part name="+3V2" library="supply1" deviceset="+3V3" device=""/>
+<part name="U1" library="bt_regulator" deviceset="LD29150" device="DT" value="LD29150DT50R"/>
+<part name="C1" library="rcl" deviceset="C-US" device="C1206" value="106"/>
 </parts>
 <sheets>
@@
 </instance>
 <instance part="U2" gate="G$1" x="228.6" y="40.64"/>
-<instance part="JP3" gate="A" x="299.72" y="55.88" rot="MR0">
-<attribute name="OC_NEWARK" x="299.72" y="55.88" size="1.778" layer="96" display="off"/>
-<attribute name="MF" x="299.72" y="55.88" size="1.778" layer="96" display="off"/>
-<attribute name="MPN" x="299.72" y="55.88" size="1.778" layer="96" display="off"/>
+<instance part="JP3" gate="A" x="304.8" y="55.88" rot="MR0">
+<attribute name="OC_NEWARK" x="304.8" y="55.88" size="1.778" layer="96" display="off"/>
+<attribute name="MF" x="304.8" y="55.88" size="1.778" layer="96" display="off"/>
+<attribute name="MPN" x="304.8" y="55.88" size="1.778" layer="96" display="off"/>
 </instance>
 <instance part="P+3" gate="1" x="314.96" y="78.74"/>
@@
 <attribute name="MPN" x="309.88" y="119.38" size="1.778" layer="96" display="off"/>
 </instance>
-<instance part="C2" gate="G$1" x="289.56" y="53.34"/>
+<instance part="C2" gate="G$1" x="292.1" y="50.8"/>
 <instance part="C4" gate="G$1" x="297.18" y="185.42" rot="R90"/>
 <instance part="C5" gate="G$1" x="297.18" y="167.64" rot="R90"/>
@@
 <instance part="+3V8" gate="G$1" x="360.68" y="71.12"/>
 <instance part="C17" gate="G$1" x="360.68" y="50.8"/>
-<instance part="IC1" gate="1" x="276.86" y="68.58"/>
-<instance part="BECSEL" gate="A" x="297.18" y="78.74"/>
+<instance part="BECSEL" gate="A" x="302.26" y="78.74"/>
 <instance part="+3V2" gate="G$1" x="132.08" y="203.2"/>
+<instance part="U1" gate="G$1" x="276.86" y="66.04"/>
+<instance part="C1" gate="G$1" x="264.16" y="50.8"/>
 </instances>
 <busses>
@@
 <segment>
 <pinref part="JP3" gate="A" pin="2"/>
-<wire x1="307.34" y1="35.56" x2="307.34" y2="55.88" width="0.1524" layer="91"/>
-<wire x1="307.34" y1="55.88" x2="302.26" y2="55.88" width="0.1524" layer="91"/>
+<wire x1="312.42" y1="35.56" x2="312.42" y2="55.88" width="0.1524" layer="91"/>
+<wire x1="312.42" y1="55.88" x2="307.34" y2="55.88" width="0.1524" layer="91"/>
 <pinref part="SUPPLY12" gate="GND" pin="GND"/>
 <wire x1="327.66" y1="33.02" x2="327.66" y2="35.56" width="0.1524" layer="91"/>
@@
 <wire x1="327.66" y1="35.56" x2="327.66" y2="45.72" width="0.1524" layer="91"/>
 <pinref part="C17" gate="G$1" pin="-"/>
-<wire x1="307.34" y1="35.56" x2="327.66" y2="35.56" width="0.1524" layer="91"/>
+<wire x1="312.42" y1="35.56" x2="327.66" y2="35.56" width="0.1524" layer="91"/>
 <wire x1="327.66" y1="35.56" x2="342.9" y2="35.56" width="0.1524" layer="91"/>
 <wire x1="342.9" y1="35.56" x2="360.68" y2="35.56" width="0.1524" layer="91"/>
@@
 <junction x="342.9" y="35.56"/>
 <pinref part="C2" gate="G$1" pin="2"/>
-<pinref part="IC1" gate="1" pin="GND"/>
 <wire x1="276.86" y1="60.96" x2="276.86" y2="35.56" width="0.1524" layer="91"/>
-<wire x1="276.86" y1="35.56" x2="289.56" y2="35.56" width="0.1524" layer="91"/>
-<junction x="307.34" y="35.56"/>
-<wire x1="289.56" y1="35.56" x2="307.34" y2="35.56" width="0.1524" layer="91"/>
-<wire x1="289.56" y1="48.26" x2="289.56" y2="35.56" width="0.1524" layer="91"/>
-<junction x="289.56" y="35.56"/>
+<wire x1="276.86" y1="35.56" x2="292.1" y2="35.56" width="0.1524" layer="91"/>
+<junction x="312.42" y="35.56"/>
+<wire x1="292.1" y1="35.56" x2="312.42" y2="35.56" width="0.1524" layer="91"/>
+<wire x1="292.1" y1="45.72" x2="292.1" y2="35.56" width="0.1524" layer="91"/>
+<junction x="292.1" y="35.56"/>
+<pinref part="U1" gate="G$1" pin="GND"/>
+<pinref part="C1" gate="G$1" pin="2"/>
+<wire x1="276.86" y1="35.56" x2="264.16" y2="35.56" width="0.1524" layer="91"/>
+<wire x1="264.16" y1="35.56" x2="264.16" y2="45.72" width="0.1524" layer="91"/>
+<junction x="276.86" y="35.56"/>
 </segment>
 <segment>
@@
 <wire x1="314.96" y1="76.2" x2="314.96" y2="68.58" width="0.1524" layer="91"/>
 <wire x1="314.96" y1="68.58" x2="314.96" y2="58.42" width="0.1524" layer="91"/>
-<wire x1="314.96" y1="58.42" x2="302.26" y2="58.42" width="0.1524" layer="91"/>
+<wire x1="314.96" y1="58.42" x2="307.34" y2="58.42" width="0.1524" layer="91"/>
 <pinref part="C2" gate="G$1" pin="1"/>
 <junction x="314.96" y="58.42"/>
-<wire x1="284.48" y1="68.58" x2="289.56" y2="68.58" width="0.1524" layer="91"/>
-<pinref part="IC1" gate="1" pin="OUT"/>
+<wire x1="284.48" y1="68.58" x2="292.1" y2="68.58" width="0.1524" layer="91"/>
 <junction x="314.96" y="68.58"/>
 <pinref part="BECSEL" gate="A" pin="3"/>
-<wire x1="289.56" y1="68.58" x2="314.96" y2="68.58" width="0.1524" layer="91"/>
-<wire x1="294.64" y1="76.2" x2="289.56" y2="76.2" width="0.1524" layer="91"/>
-<wire x1="289.56" y1="76.2" x2="289.56" y2="68.58" width="0.1524" layer="91"/>
-<junction x="289.56" y="68.58"/>
-<wire x1="289.56" y1="55.88" x2="289.56" y2="68.58" width="0.1524" layer="91"/>
+<wire x1="292.1" y1="68.58" x2="314.96" y2="68.58" width="0.1524" layer="91"/>
+<wire x1="299.72" y1="76.2" x2="292.1" y2="76.2" width="0.1524" layer="91"/>
+<wire x1="292.1" y1="76.2" x2="292.1" y2="68.58" width="0.1524" layer="91"/>
+<junction x="292.1" y="68.58"/>
+<wire x1="292.1" y1="53.34" x2="292.1" y2="68.58" width="0.1524" layer="91"/>
+<pinref part="U1" gate="G$1" pin="VOUT"/>
 </segment>
 <segment>
@@
 <segment>
 <label x="279.4" y="78.74" size="1.778" layer="95"/>
-<wire x1="294.64" y1="78.74" x2="279.4" y2="78.74" width="0.1524" layer="91"/>
+<wire x1="299.72" y1="78.74" x2="279.4" y2="78.74" width="0.1524" layer="91"/>
 <pinref part="BECSEL" gate="A" pin="2"/>
 </segment>
@@
 <net name="N$3" class="0">
 <segment>
-<pinref part="IC1" gate="1" pin="IN"/>
-<wire x1="269.24" y1="68.58" x2="266.7" y2="68.58" width="0.1524" layer="91"/>
+<wire x1="269.24" y1="68.58" x2="264.16" y2="68.58" width="0.1524" layer="91"/>
 <pinref part="BECSEL" gate="A" pin="1"/>
-<wire x1="294.64" y1="81.28" x2="266.7" y2="81.28" width="0.1524" layer="91"/>
-<wire x1="266.7" y1="81.28" x2="266.7" y2="68.58" width="0.1524" layer="91"/>
-</segment>
-</net>
+<wire x1="299.72" y1="81.28" x2="264.16" y2="81.28" width="0.1524" layer="91"/>
+<wire x1="264.16" y1="81.28" x2="264.16" y2="68.58" width="0.1524" layer="91"/>
+<pinref part="U1" gate="G$1" pin="VIN"/>
+<junction x="264.16" y="68.58"/>
+<pinref part="C1" gate="G$1" pin="1"/>
+<wire x1="264.16" y1="53.34" x2="264.16" y2="68.58" width="0.1524" layer="91"/>
+</segment>
+</net>

Commit message: Renamed VBEC net
Connections:
- net N$3 renamed VBEC
Changed lines of the file:
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@@
 </segment>
 </net>
-<net name="N$3" class="0">
+<net name="VBEC" class="0">
 <segment>
 <wire x1="269.24" y1="68.58" x2="264.16" y2="68.58" width="0.1524" layer="91"/>

Commit message: Added ISP pushbutton and pullup
Parts:
- added R11: 10K, rcl:R-US_R0603
- added S1: ISP, bt_electromech:SPST_TAC_RECT1
Connections:
- net !ISP: now also R11.1, S1.S
- net +3V3: now also R11.2
- net GND: now also S1.P
Changed lines of the file:
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@@
 <part name="U1" library="bt_regulator" deviceset="LD29150" device="DT" value="LD29150DT50R"/>
 <part name="C1" library="rcl" deviceset="C-US" device="C1206" value="106"/>
+<part name="S1" library="bt_electromech" deviceset="SPST" device="_TAC_RECT1" value="ISP"/>
+<part name="SUPPLY6" library="supply2" deviceset="GND" device=""/>
+<part name="R11" library="rcl" deviceset="R-US_" device="R0603" value="10K">
+<attribute name="MF" value=""/>
+<attribute name="MPN" value="WCR0805-220RFI"/>
+<attribute name="OC_NEWARK" value="98K2621"/>
+</part>
+<part name="+3V10" library="supply1" deviceset="+3V3" device=""/>
 </parts>
 <sheets>
@@
 </instance>
 <instance part="+3V7" gate="G$1" x="368.3" y="129.54"/>
-<instance part="SUPPLY9" gate="GND" x="157.48" y="116.84"/>
+<instance part="SUPPLY9" gate="GND" x="157.48" y="114.3"/>
 <instance part="JP28" gate="A" x="309.88" y="137.16">
 <attribute name="OC_NEWARK" x="309.88" y="137.16" size="1.778" layer="96" display="off"/>
@@
 <instance part="U1" gate="G$1" x="276.86" y="66.04"/>
 <instance part="C1" gate="G$1" x="264.16" y="50.8"/>
+<instance part="S1" gate="G$1" x="182.88" y="124.46" rot="R90"/>
+<instance part="SUPPLY6" gate="GND" x="182.88" y="114.3"/>
+<instance part="R11" gate="G$1" x="182.88" y="144.78" rot="MR90">
+<attribute name="OC_NEWARK" x="182.88" y="144.78" size="1.778" layer="96" rot="MR270" display="off"/>
+<attribute name="MF" x="182.88" y="144.78" size="1.778" layer="96" rot="MR270" display="off"/>
+<attribute name="MPN" x="182.88" y="144.78" size="1.778" layer="96" rot="MR270" display="off"/>
+</instance>
+<instance part="+3V10" gate="G$1" x="182.88" y="157.48"/>
 </instances>
 <busses>
@@
 <pinref part="U$1" gate="G$1" pin="GND2"/>
 <wire x1="124.46" y1="124.46" x2="157.48" y2="124.46" width="0.1524" layer="91"/>
-<wire x1="157.48" y1="124.46" x2="157.48" y2="119.38" width="0.1524" layer="91"/>
+<wire x1="157.48" y1="124.46" x2="157.48" y2="116.84" width="0.1524" layer="91"/>
 <pinref part="SUPPLY9" gate="GND" pin="GND"/>
+</segment>
+<segment>
+<pinref part="SUPPLY6" gate="GND" pin="GND"/>
+<pinref part="S1" gate="G$1" pin="P"/>
+<wire x1="182.88" y1="116.84" x2="182.88" y2="119.38" width="0.1524" layer="91"/>
 </segment>
 </net>
@@
 <pinref part="+3V2" gate="G$1" pin="+3V3"/>
 </segment>
+<segment>
+<pinref part="R11" gate="G$1" pin="2"/>
+<pinref part="+3V10" gate="G$1" pin="+3V3"/>
+<wire x1="182.88" y1="154.94" x2="182.88" y2="149.86" width="0.1524" layer="91"/>
+</segment>
 </net>
 <net name="SDA" class="0">
@@
 <net name="!ISP" class="0">
 <segment>
-<wire x1="124.46" y1="132.08" x2="157.48" y2="132.08" width="0.1524" layer="91"/>
+<wire x1="124.46" y1="132.08" x2="182.88" y2="132.08" width="0.1524" layer="91"/>
 <label x="157.48" y="132.08" size="1.778" layer="95" rot="MR0"/>
 <pinref part="U$1" gate="G$1" pin="P2.10"/>
-</segment>
-</net>
+<pinref part="R11" gate="G$1" pin="1"/>
+<wire x1="182.88" y1="132.08" x2="182.88" y2="139.7" width="0.1524" layer="91"/>
+<junction x="182.88" y="132.08"/>
+<pinref part="S1" gate="G$1" pin="S"/>
+<wire x1="182.88" y1="129.54" x2="182.88" y2="132.08" width="0.1524" layer="91"/>
+</segment>
+</net>
