File: RoverBaseboard/RoverBaseboard.sch (EAGLE design)
At the start: 61 parts, among them IC3 3.3V, U1 LD29150DT50R, U2 microSD

Commit message: Added ISP pin headers, revised power supply selection layout, added pin header for selecting external 5VIN in addition to selections for 5V or 6V BEC. Renumbered capacitors. Verified cap voltages, etc.
Parts:
- removed BECSEL: 5V | 6V, pinhead-2:PINHD-1X03_2.54-S
- removed C1, C2, C3: 106, rcl:C-USC1206
- removed C17: 33uF, rcl:CPOL-US140CLH-0810
- removed S1: ISP, bt_electromech:SPST_TAC_RECT1
- added BEC: BYP | REG, pinhead-2:PINHD-1X03_2.54-S
- added C40, C41, C46\: 106, rcl:C-USC0603
- added JP12: 5VIN, pinhead-2:PINHD-1X01_2.54-S
- added JP30: ISP, pinhead-2:PINHD-1X02_2.54-S
- C10: device rcl:C-USC0603 -> rcl:C-USC1206; VOLTAGE (none) -> 10V
- C11, C12: value 106 -> 33uF; device rcl:C-USC0603 -> rcl:CPOL-USSMCB
- JP3: value POWER -> PWR
- renumbered C13 to C43, C14 to C45, C15 to C47, C4 to C30, C5 to C31, C6 to C20, C7 to C21, C8 to C42, C9 to C44
Connections:
- removed net VBEC: BECSEL.1, C1.1, U1.VIN
- new net 5VIN: JP12.1, JP3.1
- new net 6-7V: BEC.1, C10.1, U1.VIN
- net !ISP: now also JP30.1; no longer S1.S
- net +3V3: now also C12.+, C41.1; no longer C12.1, C17.+
- net +5V: now also BEC.3, C11.+, C40.1, C46\.1; no longer BECSEL.3, C10.1, C11.1, C2.1, C3.1, JP3.1
- net BEC: now also BEC.2; no longer BECSEL.2
- net GND: now also C11.-, C12.-, C40.2, C41.2, C46\.2, JP30.2; no longer C1.2, C11.2, C12.2, C17.-, C2.2, C3.2, S1.P
Other:
- note removed: "Verify input cap values"
- moved on the sheet: C10, IC3, JP3, R11, U1

Commit message: Added documentation to schematic
Parts:
- BEC: value BYP | REG -> REG | BYP | 5VIN
Other:
- note added: "Select power source"
Changed lines of the file:
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@@
 <part name="+3V8" library="supply1" deviceset="+3V3" device=""/>
 <part name="C12" library="rcl" deviceset="CPOL-US" device="SMCB" value="33uF"/>
-<part name="BEC" library="pinhead-2" deviceset="PINHD-1X03" device="_2.54-S" value="BYP | REG"/>
+<part name="BEC" library="pinhead-2" deviceset="PINHD-1X03" device="_2.54-S" value="REG | BYP | 5VIN"/>
 <part name="+3V2" library="supply1" deviceset="+3V3" device=""/>
 <part name="U1" library="bt_regulator" deviceset="LD29150" device="DT" value="LD29150DT50R"/>
@@
 <text x="76.2" y="208.28" size="2.54" layer="97">LPXpresso / MBED</text>
 <text x="302.26" y="88.9" size="1.778" layer="97">POWER SUPPLY</text>
+<text x="248.92" y="63.5" size="1.778" layer="97" rot="R90">Select power source</text>
 </plain>
 <instances>

Commit message: Revised net names to better reflect encoders. Changed pin header labels to better reflect function.
Parts:
- JP1: value IO -> D0
- JP10: value PWM -> P1
- JP11: value PWM -> P2
- JP13: value IO -> D1
- JP14: value DIGITAL -> D2
- JP15: value ENCODERS -> A
- JP16: value ADC -> A0
- JP17: value ADC -> A1
- JP18: value ADC -> A2
- JP19: value ADC -> A3
- JP2: value ENCODERS -> B
- JP28: value DIGITAL -> D7
- JP29: value DIGITAL -> D8
Connections:
- net ENC0 renamed ENCA_LEFT
- net ENC1 renamed ENCA_RIGHT
- net ENC2 renamed ENCB_RIGHT
- net ENC3 renamed ENCB_LEFT
Changed lines of the file:
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@@
 <part name="+3V1" library="supply1" deviceset="+3V3" device=""/>
 <part name="SUPPLY1" library="supply2" deviceset="GND" device=""/>
-<part name="JP15" library="pinhead-2" deviceset="PINHD-1X04" device="_2.54-S" value="ENCODERS">
+<part name="JP15" library="pinhead-2" deviceset="PINHD-1X04" device="_2.54-S" value="A">
 <attribute name="MF" value=""/>
 <attribute name="MPN" value=""/>
@@
 </part>
 <part name="P+5" library="supply1" deviceset="+5V" device=""/>
-<part name="JP2" library="pinhead-2" deviceset="PINHD-1X04" device="_2.54-S" value="ENCODERS">
+<part name="JP2" library="pinhead-2" deviceset="PINHD-1X04" device="_2.54-S" value="B">
 <attribute name="MF" value=""/>
 <attribute name="MPN" value=""/>
@@
 <attribute name="OC_NEWARK" value="unknown"/>
 </part>
-<part name="JP10" library="pinhead-2" deviceset="PINHD-1X03" device="_2.54-S" value="PWM">
-<attribute name="MF" value=""/>
-<attribute name="MPN" value=""/>
-<attribute name="OC_NEWARK" value="unknown"/>
-</part>
-<part name="JP11" library="pinhead-2" deviceset="PINHD-1X03" device="_2.54-S" value="PWM">
+<part name="JP10" library="pinhead-2" deviceset="PINHD-1X03" device="_2.54-S" value="P1">
+<attribute name="MF" value=""/>
+<attribute name="MPN" value=""/>
+<attribute name="OC_NEWARK" value="unknown"/>
+</part>
+<part name="JP11" library="pinhead-2" deviceset="PINHD-1X03" device="_2.54-S" value="P2">
 <attribute name="MF" value=""/>
 <attribute name="MPN" value=""/>
@@
 <part name="SUPPLY5" library="supply2" deviceset="GND" device=""/>
 <part name="SUPPLY10" library="supply2" deviceset="GND" device=""/>
-<part name="JP1" library="pinhead-2" deviceset="PINHD-1X03" device="_2.54-S" value="IO">
+<part name="JP1" library="pinhead-2" deviceset="PINHD-1X03" device="_2.54-S" value="D0">
 <attribute name="MF" value=""/>
 <attribute name="MPN" value=""/>
@@
 </part>
 <part name="+3V6" library="supply1" deviceset="+3V3" device=""/>
-<part name="JP13" library="pinhead-2" deviceset="PINHD-1X03" device="_2.54-S" value="IO">
-<attribute name="MF" value=""/>
-<attribute name="MPN" value=""/>
-<attribute name="OC_NEWARK" value="unknown"/>
-</part>
-<part name="JP14" library="pinhead-2" deviceset="PINHD-1X03" device="_2.54-S" value="DIGITAL">
+<part name="JP13" library="pinhead-2" deviceset="PINHD-1X03" device="_2.54-S" value="D1">
+<attribute name="MF" value=""/>
+<attribute name="MPN" value=""/>
+<attribute name="OC_NEWARK" value="unknown"/>
+</part>
+<part name="JP14" library="pinhead-2" deviceset="PINHD-1X03" device="_2.54-S" value="D2">
 <attribute name="MF" value=""/>
 <attribute name="MPN" value=""/>
@@
 </part>
 <part name="U$1" library="LPCXpresso" deviceset="LPCXPRESSO_NO_PAD" device="_1768_REVB" value="LPCXPRESSO"/>
-<part name="JP16" library="pinhead-2" deviceset="PINHD-1X03" device="_2.54-S" value="ADC">
-<attribute name="MF" value=""/>
-<attribute name="MPN" value=""/>
-<attribute name="OC_NEWARK" value="unknown"/>
-</part>
-<part name="JP17" library="pinhead-2" deviceset="PINHD-1X03" device="_2.54-S" value="ADC">
-<attribute name="MF" value=""/>
-<attribute name="MPN" value=""/>
-<attribute name="OC_NEWARK" value="unknown"/>
-</part>
-<part name="JP18" library="pinhead-2" deviceset="PINHD-1X03" device="_2.54-S" value="ADC">
-<attribute name="MF" value=""/>
-<attribute name="MPN" value=""/>
-<attribute name="OC_NEWARK" value="unknown"/>
-</part>
-<part name="JP19" library="pinhead-2" deviceset="PINHD-1X03" device="_2.54-S" value="ADC">
+<part name="JP16" library="pinhead-2" deviceset="PINHD-1X03" device="_2.54-S" value="A0">
+<attribute name="MF" value=""/>
+<attribute name="MPN" value=""/>
+<attribute name="OC_NEWARK" value="unknown"/>
+</part>
+<part name="JP17" library="pinhead-2" deviceset="PINHD-1X03" device="_2.54-S" value="A1">
+<attribute name="MF" value=""/>
+<attribute name="MPN" value=""/>
+<attribute name="OC_NEWARK" value="unknown"/>
+</part>
+<part name="JP18" library="pinhead-2" deviceset="PINHD-1X03" device="_2.54-S" value="A2">
+<attribute name="MF" value=""/>
+<attribute name="MPN" value=""/>
+<attribute name="OC_NEWARK" value="unknown"/>
+</part>
+<part name="JP19" library="pinhead-2" deviceset="PINHD-1X03" device="_2.54-S" value="A3">
 <attribute name="MF" value=""/>
 <attribute name="MPN" value=""/>
@@
 <part name="+3V7" library="supply1" deviceset="+3V3" device=""/>
 <part name="SUPPLY9" library="supply2" deviceset="GND" device=""/>
-<part name="JP28" library="pinhead-2" deviceset="PINHD-1X03" device="_2.54-S" value="DIGITAL">
-<attribute name="MF" value=""/>
-<attribute name="MPN" value=""/>
-<attribute name="OC_NEWARK" value="unknown"/>
-</part>
-<part name="JP29" library="pinhead-2" deviceset="PINHD-1X03" device="_2.54-S" value="DIGITAL">
+<part name="JP28" library="pinhead-2" deviceset="PINHD-1X03" device="_2.54-S" value="D7">
+<attribute name="MF" value=""/>
+<attribute name="MPN" value=""/>
+<attribute name="OC_NEWARK" value="unknown"/>
+</part>
+<part name="JP29" library="pinhead-2" deviceset="PINHD-1X03" device="_2.54-S" value="D8">
 <attribute name="MF" value=""/>
 <attribute name="MPN" value=""/>
@@
 </segment>
 </net>
-<net name="ENC2" class="0">
+<net name="ENCB_RIGHT" class="0">
 <segment>
 <pinref part="JP2" gate="A" pin="2"/>
-<wire x1="71.12" y1="55.88" x2="53.34" y2="55.88" width="0.1524" layer="91"/>
-<label x="53.34" y="55.88" size="1.778" layer="95"/>
+<wire x1="71.12" y1="55.88" x2="43.18" y2="55.88" width="0.1524" layer="91"/>
+<label x="43.18" y="55.88" size="1.778" layer="95"/>
 </segment>
 <segment>
@@
 </segment>
 </net>
-<net name="ENC3" class="0">
+<net name="ENCB_LEFT" class="0">
 <segment>
 <pinref part="JP2" gate="A" pin="3"/>
-<wire x1="71.12" y1="53.34" x2="53.34" y2="53.34" width="0.1524" layer="91"/>
-<label x="53.34" y="53.34" size="1.778" layer="95"/>
+<wire x1="71.12" y1="53.34" x2="43.18" y2="53.34" width="0.1524" layer="91"/>
+<label x="43.18" y="53.34" size="1.778" layer="95"/>
 </segment>
 <segment>
@@
 </segment>
 </net>
-<net name="ENC0" class="0">
+<net name="ENCA_LEFT" class="0">
 <segment>
 <pinref part="U$1" gate="G$1" pin="P0.4/CAN_RX2"/>
@@
 <segment>
 <pinref part="JP15" gate="A" pin="3"/>
-<wire x1="71.12" y1="73.66" x2="53.34" y2="73.66" width="0.1524" layer="91"/>
-<label x="53.34" y="73.66" size="1.778" layer="95"/>
-</segment>
-</net>
-<net name="ENC1" class="0">
+<wire x1="71.12" y1="73.66" x2="43.18" y2="73.66" width="0.1524" layer="91"/>
+<label x="43.18" y="73.66" size="1.778" layer="95"/>
+</segment>
+</net>
+<net name="ENCA_RIGHT" class="0">
 <segment>
 <pinref part="U$1" gate="G$1" pin="P0.5/CAN_TX2"/>
@@
 <segment>
 <pinref part="JP15" gate="A" pin="2"/>
-<wire x1="71.12" y1="76.2" x2="53.34" y2="76.2" width="0.1524" layer="91"/>
-<label x="53.34" y="76.2" size="1.778" layer="95"/>
-</segment>
-</net>
+<wire x1="71.12" y1="76.2" x2="43.18" y2="76.2" width="0.1524" layer="91"/>
+<label x="43.18" y="76.2" size="1.778" layer="95"/>
+</segment>
+</net>

Commit message: Updated pin names, removed BEC>5V regulator, moved VIN pins back to original spot.
Parts:
- removed BEC: REG | BYP | 5VIN, pinhead-2:PINHD-1X03_2.54-S
- removed C10: 106, rcl:C-USC1206
- removed JP12: 5VIN, pinhead-2:PINHD-1X01_2.54-S
- removed U1: LD29150DT50R, bt_regulator:LD29150DT
- C11, C12: value 33uF -> 10uF; device rcl:CPOL-USSMCB -> rcl:C-USC1206
- JP3: value PWR -> POWER
Connections:
- net D0 renamed P11
- net D1 renamed P12
- removed net 5VIN: JP12.1, JP3.1
- removed net 6-7V: BEC.1, C10.1, U1.VIN
- net +3V3: now also C12.1; no longer C12.+
- net +5V: now also C11.1, JP3.1; no longer BEC.3, C11.+, U1.VOUT
- net BEC: no longer BEC.2
- net GND: now also C11.2, C12.2; no longer C10.2, C11.-, C12.-, U1.GND
Other:
- note removed: "Select power source"
- moved on the sheet: JP3
